File: pcb/tv-side-keyboard.kicad_pcb (KiCad board)
At the start: 2 copper layers, 117 x 68 mm, 51 parts, among them J1 ESP-Prog-ProgramCOM-RECV, SW1 SW_Push, SW10 SW_Push, SW11 SW_Push, SW12 SW_Push, SW2 SW_Push, SW3 SW_Push, SW4 SW_Push, SW5 SW_Push, SW6 SW_Push, SW7 SW_Push, SW8 SW_Push, SW9 SW_Push, U1 M5StampS3, U2 M5 IR Unit

Commit message: build-pcb
Parts:
- moved R1 2.70 mm to (59.3, 59.1)
- moved R2 2.70 mm to (57.3, 59.1)
- moved R3 1.30 mm to (87.1, 38.3)
- turned J1 to 180 degrees
Routing:
- net +5V: track 0.00 -> 401.5 mm
- net +3V3: track 0.00 -> 65.3 mm

Commit message: build-pcb
Parts:
- moved H2 1.00 mm to (57.0, 34.0)
- moved H7 1.00 mm to (57.0, 94.0)
Routing:
- added copper zone on B.Cu, net GND
- added copper zone on F.Cu, net GND
Other:
- board size 117 x 68 mm -> 118 x 68 mm
Changed lines of the file:
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@@
   )
   (footprint "$sparrow62:M2_v2" (layer "F.Cu")
-    (at 58 94)
+    (at 57 94)
     (attr through_hole)
     (fp_text reference "H7" (at 0 1.905) (layer "Dwgs.User") hide
@@
   )
   (footprint "$sparrow62:M2_v2" (layer "F.Cu")
-    (at 58 34)
+    (at 57 34)
     (attr through_hole)
     (fp_text reference "H2" (at 0 1.905) (layer "Dwgs.User") hide
@@
   (gr_arc (start 171 93) (mid 169.535534 96.535534) (end 166 98)
     (stroke (width 0.1) (type default)) (layer "Edge.Cuts"))
-  (gr_arc (start 54 35) (mid 55.464466 31.464466) (end 59 30)
+  (gr_arc (start 53 35) (mid 54.464466 31.464466) (end 58 30)
     (stroke (width 0.1) (type default)) (layer "Edge.Cuts"))
-  (gr_arc (start 59 98) (mid 55.464466 96.535534) (end 54 93)
+  (gr_arc (start 58 98) (mid 54.464466 96.535534) (end 53 93)
     (stroke (width 0.1) (type default)) (layer "Edge.Cuts"))
-  (gr_line (start 59 30) (end 166 30)
+  (gr_line (start 58 30) (end 166 30)
     (stroke (width 0.1) (type default)) (layer "Edge.Cuts"))
-  (gr_line (start 54 93) (end 54 35)
+  (gr_line (start 53 93) (end 53 35)
     (stroke (width 0.1) (type default)) (layer "Edge.Cuts"))
   (gr_arc (start 166 30) (mid 169.535534 31.464466) (end 171 35)
     (stroke (width 0.1) (type default)) (layer "Edge.Cuts"))
-  (gr_line (start 166 98) (end 59 98)
+  (gr_line (start 166 98) (end 58 98)
     (stroke (width 0.1) (type default)) (layer "Edge.Cuts"))
   (gr_line (start 171 35) (end 171 93)
@@
   (segment (start 106.2 60.9) (end 107.4 59.7) (width 0.25) (layer "B.Cu") (net 15))
   (segment (start 103 79.9) (end 101.5 78.4) (width 0.25) (layer "B.Cu") (net 15))
+  (zone (net 4) (net_name "GND") (layers "F&B.Cu") (hatch edge 0.5)
+    (connect_pads (clearance 0.5))
+    (min_thickness 0.25) (filled_areas_thickness no)
+    (fill yes (thermal_gap 0.5) (thermal_bridge_width 0.5))
+    (polygon
+      (pts
+        (xy 51 24)
+        (xy 174 24)
+        (xy 174 103)
+        (xy 51 103)
+      )
+    )
+  )
 )

Commit message: v1.0.0
Parts:
- added G***: LOGO, $74th:74th-10mm, B.Cu at (79.9, 87.9)
- added REF**: JLCJLCJLCJLC, $74th:JLCJLCJLCJLC, B.Cu at (69.0, 34.8)
- G***: footprint $sparrow62:Sparrow2 -> $sparrow62:Sparrow2_oneside
- moved CH1 3.31 mm to (55.0, 83.5)
- moved G*** 2.12 mm to (64.3, 82.9)
- renumbered U2 to CH2, D4 to D1, D11 to D10, D10 to D11, D16 to D13, D15 to D14, D14 to D15, D13 to D16, D20 to D17, D19 to D18, D18 to D19, D1 to D2, D17 to D20, D24 to D22, D22 to D24, D2 to D3, D3 to D4, D8 to D5, D5 to D6, D6 to D7, D7 to D8, H2 to H1, H3 to H2, H4 to H3, H1 to H4, H7 to H5, H5 to H6, H6 to H7, R3 to R1, R1 to R2, R2 to R3, SW6 to SW10, SW9 to SW11, SW4 to SW2, SW7 to SW3, SW10 to SW4, SW2 to SW5, SW5 to SW6, SW8 to SW7, SW11 to SW8, SW3 to SW9
Routing:
- net /ROW3: track 0.00 -> 171.6 mm
- net /COL2: track 0.00 -> 135.4 mm, vias 0 -> 1
- net /COL3: track 0.00 -> 133.7 mm, vias 0 -> 2
- net /COL4: track 0.00 -> 108.8 mm, vias 0 -> 4
- net /ROW2: track 0.00 -> 106.3 mm, vias 0 -> 4
- net /ROW1: track 0.00 -> 103.9 mm, vias 0 -> 4
- net Net-(D13-DOUT): track 0.00 -> 86.2 mm, vias 0 -> 2
- net /COL1: track 0.00 -> 85.7 mm, vias 0 -> 2
- net Net-(D17-DOUT): track 0.00 -> 83.7 mm, vias 0 -> 2
- net Net-(D4-A): track 0.00 -> 72.1 mm, vias 0 -> 2
- net Net-(D11-A): track 0.00 -> 61.6 mm
- net Net-(D1-A): track 0.00 -> 44.1 mm, vias 0 -> 2
- net /SCL: track 0.00 -> 44.0 mm, vias 0 -> 1
- net /SDA: track 0.00 -> 41.1 mm, vias 0 -> 1
- net Net-(D9-A): track 0.00 -> 35.1 mm
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Other:
- board text added: "@74th"
- board text added: "ESP-Prog"
- board text added: "JoyPoint"
- board text added: "M5 IR"
- board text added: "SparrowTV"
- board text added: "v1.0.0-M5StampS3"
