File: pcb/tv-side-keyboard.kicad_sch (KiCad schematic)
At the start: 43 parts, among them J1 ESP-Prog-ProgramCOM-RECV, SW1 SW_Push, SW10 SW_Push, SW11 SW_Push, SW12 SW_Push, SW2 SW_Push, SW3 SW_Push, SW4 SW_Push, SW5 SW_Push, SW6 SW_Push, SW7 SW_Push, SW8 SW_Push, SW9 SW_Push, U1 M5StampS3, U2 M5 IR Unit

Commit message: v1.0.0
Parts:
- renumbered U2 to CH2, D4 to D1, D11 to D10, D10 to D11, D16 to D13, D15 to D14, D14 to D15, D13 to D16, D20 to D17, D19 to D18, D18 to D19, D1 to D2, D17 to D20, D24 to D22, D22 to D24, D2 to D3, D3 to D4, D8 to D5, D5 to D6, D6 to D7, D7 to D8, R3 to R1, R1 to R2, R2 to R3, SW6 to SW10, SW9 to SW11, SW4 to SW2, SW7 to SW3, SW10 to SW4, SW2 to SW5, SW5 to SW6, SW8 to SW7, SW11 to SW8, SW3 to SW9
