File: pcb-kicad/tv-side-keyboard.kicad_sch (KiCad schematic)
At the start: 43 parts, among them J1 ESP-Prog-ProgramCOM-RECV, SW1 SW_Push, SW10 SW_Push, SW11 SW_Push, SW12 SW_Push, SW2 SW_Push, SW3 SW_Push, SW4 SW_Push, SW5 SW_Push, SW6 SW_Push, SW7 SW_Push, SW8 SW_Push, SW9 SW_Push, U1 M5StampS3

Commit message: update kicad
Other:
- note added: "Button Matrix"
- note added: "I2C Pointer Device Port"
- note added: "IR Unit Port"
- note added: "LEDs"
- note added: "M5StampS3"
- note added: "Program Port"
- moved on the sheet: CH1, CH2, D1, D10, D11, D12, D13, D14, D15, D16, D17, D18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

Commit message: update README
Parts:
- J1: value ESP-Prog-ProgramCOM-RECV -> ESPProg-Port
Changed lines of the file:
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@@
       (effects (font (size 1.27 1.27)))
     )
-    (property "Value" "ESP-Prog-ProgramCOM-RECV" (at 363.22 55.88 0)
+    (property "Value" "ESPProg-Port" (at 363.22 55.88 0)
       (effects (font (size 1.27 1.27)))
     )

Commit message: update BOM
Parts:
- D1, D10, D11, D12, D2, D3, D4, D5, D6, D7, D8, D9: value D -> 1N4148W
Changed lines of the file:
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@@
       (effects (font (size 1.27 1.27)) (justify right))
     )
-    (property "Value" "D" (at 83.82 167.64 90)
+    (property "Value" "1N4148W" (at 83.82 167.64 90)
       (effects (font (size 1.27 1.27)) (justify right))
     )
@@
       (effects (font (size 1.27 1.27)) (justify right))
     )
-    (property "Value" "D" (at 151.13 191.77 90)
+    (property "Value" "1N4148W" (at 151.13 191.77 90)
       (effects (font (size 1.27 1.27)) (justify right))
     )
@@
       (effects (font (size 1.27 1.27)) (justify right))
     )
-    (property "Value" "D" (at 128.27 217.17 90)
+    (property "Value" "1N4148W" (at 128.27 217.17 90)
       (effects (font (size 1.27 1.27)) (justify right))
     )
@@
       (effects (font (size 1.27 1.27)) (justify right))
     )
-    (property "Value" "D" (at 128.27 191.77 90)
+    (property "Value" "1N4148W" (at 128.27 191.77 90)
       (effects (font (size 1.27 1.27)) (justify right))
     )
@@
       (effects (font (size 1.27 1.27)) (justify right))
     )
-    (property "Value" "D" (at 106.68 217.17 90)
+    (property "Value" "1N4148W" (at 106.68 217.17 90)
       (effects (font (size 1.27 1.27)) (justify right))
     )
@@
       (effects (font (size 1.27 1.27)) (justify right))
     )
-    (property "Value" "D" (at 151.13 167.64 90)
+    (property "Value" "1N4148W" (at 151.13 167.64 90)
       (effects (font (size 1.27 1.27)) (justify right))
     )
@@
       (effects (font (size 1.27 1.27)) (justify right))
     )
-    (property "Value" "D" (at 83.82 217.17 90)
+    (property "Value" "1N4148W" (at 83.82 217.17 90)
       (effects (font (size 1.27 1.27)) (justify right))
     )
@@
       (effects (font (size 1.27 1.27)) (justify right))
     )
-    (property "Value" "D" (at 106.68 167.64 90)
+    (property "Value" "1N4148W" (at 106.68 167.64 90)
       (effects (font (size 1.27 1.27)) (justify right))
     )
@@
       (effects (font (size 1.27 1.27)) (justify right))
     )
-    (property "Value" "D" (at 83.82 191.77 90)
+    (property "Value" "1N4148W" (at 83.82 191.77 90)
       (effects (font (size 1.27 1.27)) (justify right))
     )
@@
       (effects (font (size 1.27 1.27)) (justify right))
     )
-    (property "Value" "D" (at 151.13 217.17 90)
+    (property "Value" "1N4148W" (at 151.13 217.17 90)
       (effects (font (size 1.27 1.27)) (justify right))
     )
@@
       (effects (font (size 1.27 1.27)) (justify right))
     )
-    (property "Value" "D" (at 128.27 167.64 90)
+    (property "Value" "1N4148W" (at 128.27 167.64 90)
       (effects (font (size 1.27 1.27)) (justify right))
     )
@@
       (effects (font (size 1.27 1.27)) (justify right))
     )
-    (property "Value" "D" (at 106.68 191.77 90)
-      (effects (font (size 1.27 1.27)) (justify right))
-    )
+    (property "Value" "1N4148W" (at 106.68 191.77 90)
+      (effects (font (size 1.27 1.27)) (justify right))
+    )

Commit message: update README
Other:
- title: (none) -> SparrowTV
Changed lines of the file:
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@@
 (kicad_sch (version 20230121) (generator eeschema)
   (paper "A3")
+  (title_block
+    (title "SparrowTV")
+  )
   (junction (at 125.73 219.71) (diameter 0) (color 0 0 0 0)
   )

Commit message: v1.1.0
Parts:
- removed CH1: JoyPoint, $74th:HY2.0_Socket_SMD_4Pin, symbol $74th:I2C_Grove_Device
- removed U1: M5StampS3, $74th-imported:STAMP-S3-DIP, symbol $74th:M5StampS3
- added C1 (x2), C11, C13, C2 (x2), C4, C6: 100n, $74th:Capacitor_0805_2012, symbol Device:C
- added C12, C3, C7: 1u, $74th:Capacitor_0805_2012, symbol Device:C
- added C5, C8: 10u, $74th:Capacitor_0805_2012, symbol Device:C
- added CH2: Grove I2C, $74th:HY2.0_Socket_SMD_4Pin, symbol $74th:I2C_Grove_HostSide
- added CH3: SWD 1Wire & UART TX, $74th:CH32V003-DebugPort, symbol $74th:CH32V003-DubugPort
- added J2: ESPProg-Port, $74th:6Pin, symbol $74th:ESP-Prog-ProgramCOM-RECV-Straight
- added J3: Keyboard USB, $74th:USB-C-12-Pin-SMD, symbol $74th:USB2.0_C_v3
- added R10, R11: 1k, $74th:Register_0805_2012, symbol Device:R
- added R6, R7: 5.1k, $74th:Register_0805_2012, symbol Device:R
- added R7, R8: 10k, $74th:Register_0805_2012, symbol Device:R
- added R8: 42k, $74th:Register_0805_2012, symbol Device:R
- added R9: 1, $74th:Register_0805_2012, symbol Device:R
- added U1: joystick-b10k, $74th:JOYSTICK-B10K, symbol $74th:joystick-b10k
- added U2: ESP32-C3-WROOM-02, $74th-imported:ESP32-C3-WROOM-02, symbol $74th:ESP32-C3-WROOM-02
- added U3: CH217K, Package_TO_SOT_SMD:SOT-23-6, symbol $74th:CH217K-USB_Power_Limit_Switch
- added U4: CH9329, Package_SO:SOIC-16_3.9x9.9mm_P1.27mm, symbol $74th:CH9329
- added U5: Regulator_AMS117-3.3, Package_TO_SOT_SMD:SOT-223-3_TabPin2, symbol $74th:Regulator_AMS117-3.3_SOT223
- added U6: CH32V003F4P6, Package_SO:TSSOP-20_4.4x6.5mm_P0.65mm, symbol $74th:CH32V003F4P6
- R1, R2, R3: footprint $74th:Capacitor_0805_2012 -> $74th:Register_0805_2012
- renumbered CH2 to CH1, SW4 to SW10, SW8 to SW11, SW5 to SW2, SW9 to SW3, SW2 to SW4, SW6 to SW5, SW10 to SW6, SW3 to SW7, SW7 to SW8, SW11 to SW9
Connections:
- net +5V: now also C5.1, C6.1, C7.1, J2.1 (VCC), U3.1 (VOUT), U4.15 (VCC), U5.3 (VI); no longer D13.1 (VDD), D14.1 (VDD), D15.1 (VDD), D16.1 (VDD), D17.1 (VDD), D18.1 (VDD), D19.1 (VDD), D20.1 (VDD), D21.1 (VDD), D22.1 (VDD), D23.1 (VDD), D24.1 (VDD)
- net COL1: now also U6.1 (PD4/UART_CK/ADC7)
- net COL2: now also U6.3 (PD6/UART_RX/ADC6)
- net COL3: now also U6.8 (PD0)
- net COL4: now also U6.10 (PC0)
- net GND: now also C1.2, C1.2, C11.2, C12.2, C13.2, C2.2, C2.2, C3.2, C4.2, C5.2, C6.2, C7.2, C8.2, CH2.4 (GND), CH3.2 (GND), J2.2 (GND), J3.4 (GND), R6.2, R7.2, R7.2, R8.2, U1.3 (XIN2), U1.6 (YIN2), U2.19 (GND), U2.9 (GND), U3.2 (GND), U4.14 (GND), U5.1 (GND), U6.7 (VSS)
- net IR_IN: now also U2.18 (GPIO0/ADC1_CH0/XTAL_32K_P)
- net IR_OUT: now also U2.17 (GPIO1/ADC1_CH1/XTAL_32K_N)
- net LED: now also U2.3 (GPIO4/ADC1_CH4)
- net ROW1: now also U6.17 (PC7/SPI_MISO)
- net ROW2: now also U6.19 (PD2/ADC3)
- net ROW3: now also U6.20 (PD3/UART_CTS/ADC4)
- net SCL: now also CH2.1 (SCL), R11.2, U2.15 (GPIO3/ADC1_CH3), U6.12 (PC2/I2C_SCL/UART_RTS); no longer R3.2
- net SDA: now also CH2.2 (SDA), R10.2, U2.16 (GPIO2/ADC1_CH2), U6.11 (PC1/I2C_SDA/SPI_NSS); no longer R2.2
- net +3V3 renamed +3.3V
- net +3.3V: now also D13.1 (VDD), D14.1 (VDD), D15.1 (VDD), D16.1 (VDD), D17.1 (VDD), D18.1 (VDD), D19.1 (VDD), D20.1 (VDD), D21.1 (VDD), D22.1 (VDD), D23.1 (VDD), D24.1 (VDD), C1.1, C1.1, C11.1, C12.1, C13.1, C2.1, C2.1, C3.1, C8.1, CH2.3 (VCC), R10.1, R11.1, R8.1, R9.1, U1.1 (XIN1), U1.4 (YIN1), U2.1 (3V3), U5.2 (VO), U6.9 (VDD)
- net BOOT renamed ESP32C3_BOOT
- net ESP32C3_BOOT: now also J2.5 (IO0), U2.8 (GPIO9)
- net EN renamed ESP32C3_RST
- net ESP32C3_RST: now also R3.2, J2.6 (EN), U2.2 (EN/CHIP_PU)
- net RXD renamed CH9329_TXD
- net CH9329_TXD: now also J2.4 (RXD0), U2.11 (GPIO20/U0RXD), U4.7 (TXD)
- net TXD renamed CH9329_RXD
- net CH9329_RXD: now also J2.3 (TXD0), U2.12 (GPIO21/U0TXD), U4.8 (RXD)
- new net: C4.1, U4.16 (V33)
- new net: J3.6 (CC2), R7.1
- new net: J3.5 (CC1), R6.1
- new net: R9.2, U6.14 (PC4/ADC2)
- new net: R7.1, U3.4 (EN#)
- new net: R8.2, U6.4 (PD7/NRST)
- new net: R2.2, U2.7 (GPIO8)
- new net: R8.1, U3.5 (ISET)
- new net CH32V003_SWDIO: CH3.1 (SWDIO), U6.18 (SWIO/PD1)
- new net CH32V003_TXD: CH3.3 (TXD), U6.2 (PD5/UART_TX/ADC5)
- new net CH9329_DM: J3.2 (D-), U4.13 (UD-)
- new net CH9329_DP: J3.3 (D+), U4.12 (UD+)
- new net VBUS: J3.1 (VBUS), U3.6 (VIN)
- new net XOUT: U1.2 (XOUT), U6.6 (PA2/ADC0/OSC_OUT)
- new net YOUT: U1.5 (YOUT), U6.5 (PA1/ADC1/OSC_IN)
- no-connect marks 9 -> 20
Other:
- note added: "CH32V003 Program Port"
- note added: "ESP32C3 Program Port"
- note added: "I2C Port"
- note added: "JoyStick"
- note added: "Main MCU"
- note added: "Sub MCU"
- note added: "USB & Power"
- note added: "USB ESP32C3"
- note added: "USB HID"
- note removed: "I2C Pointer Device Port"
- note removed: "M5StampS3"
- note removed: "Program Port"
- moved on the sheet: CH1, D1, D10, D11, D12, D13, D14, D15, D16, D17, D18, D19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

Commit message: wip
Parts:
- removed CH2: Grove I2C, $74th:HY2.0_Socket_SMD_4Pin, symbol $74th:I2C_Grove_HostSide
- added D25, D26, D27: 1N4148W, $sparrow62:D3_SMD_v2, symbol Device:D
- added D28, D29, D30: SK6812MINI, $74th:YS-SK6812MINI-E-BACK-RIGHT, symbol $74th:SK6812MINI
- added SW13, SW14, SW15: SW_Push, $sparrow62:Choc_1Side_1.0u, symbol Switch:SW_Push
- J1: renamed from J3; footprint $74th:USB-C-12-Pin-SMD -> $74th:USB-C-12-Pin-MidMount-ali-v5
- renumbered C4 to C1, C3 to C11, C2 to C12, C1 to C13, C7 to C2, C11 to C3, C12 to C4, C6 to C5, C13 to C6, C8 to C7, C5 to C8, CH3 to CH2, J1 to J2, J2 to J3, R9 to R1, R11 to R10, R10 to R11, R1 to R2, R8 to R3, R3 to R9, U6 to U2, U4 to U3, U5 to U4, U3 to U5, U2 to U6
Connections:
- net +3.3V: now also D28.1 (VDD), D29.1 (VDD), D30.1 (VDD)
- net CH9329_RXD: now also U6.6 (GPIO7); no longer J2.3 (TXD0), J3.3 (TXD0), U6.12 (GPIO21/U0TXD)
- net CH9329_TXD: now also U6.5 (GPIO6); no longer J2.5 (RXD0), J3.4 (RXD0), U6.11 (GPIO20/U0RXD)
- net COL1: now also U2.10 (PC0), SW13.1, SW14.1, SW15.1; no longer SW1.1, SW5.1, SW9.1, U2.1 (PD4/UART_CK/ADC7)
- net COL2: now also SW1.1, SW5.1, SW9.1, U2.19 (PD2/ADC3); no longer SW10.1, SW2.1, SW6.1, U2.3 (PD6/UART_RX/ADC6)
- net COL3: now also SW10.1, SW2.1, SW6.1, U2.17 (PC7/SPI_MISO); no longer SW11.1, SW3.1, SW7.1, U2.8 (PD0)
- net COL4: now also SW11.1, SW3.1, SW7.1, U2.16 (PC6/SPI_MOSI); no longer SW12.1, SW4.1, SW8.1, U2.10 (PC0)
- net GND: now also D28.3 (GND), D29.3 (GND), D30.3 (GND)
- net ROW1: now also U2.20 (PD3/UART_CTS/ADC4), D25.1 (K); no longer U2.17 (PC7/SPI_MISO)
- net ROW2: now also U2.1 (PD4/UART_CK/ADC7), D26.1 (K); no longer U2.19 (PD2/ADC3)
- net ROW3: now also U2.3 (PD6/UART_RX/ADC6), D27.1 (K); no longer U2.20 (PD3/UART_CTS/ADC4)
- net at R2.1: now also D28.4 (DIN); no longer D16.4 (DIN)
- net at D17.2 (DOUT): now also D30.4 (DIN); no longer D21.4 (DIN)
- net COL5: now reaches U2.15 (PC5/SPI_SCK)
- net COL5: now also SW12.1, SW4.1, SW8.1
- net at D20.4 (DIN): now also D29.2 (DOUT); no longer D13.2 (DOUT)
- new net: D16.4 (DIN), D28.2 (DOUT)
- new net: D13.2 (DOUT), D29.4 (DIN)
- new net: D25.2 (A), SW13.2
- new net: D26.2 (A), SW14.2
- new net: D21.4 (DIN), D30.2 (DOUT)
- new net: D27.2 (A), SW15.2
- new net ESP32C3_RXD: J2.5 (RXD0), J3.4 (RXD0), U6.11 (GPIO20/U0RXD)
- new net ESP32C3_TXD: J2.3 (TXD0), J3.3 (TXD0), U6.12 (GPIO21/U0TXD)
- no-connect marks 20 -> 17
Other:
- note removed: "I2C Port"
- note removed: "USB ESP32C3"
- moved on the sheet: CH1, D1, D10, D11, D12, D13, D14, D15, D16, D17, D18, D19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

Commit message: iphone se 2 sized
Parts:
- CH2: footprint $74th:CH32V003-DebugPort -> 74th:PinOut_4Pin; symbol $74th:CH32V003-DubugPort -> 74th_Interface:SWD_WCH-1Wire_WITH-TXD-VCC
- renumbered C7 to C1, C8 to C2, C6 to C3, C3 to C4, C4 to C5, C5 to C6, C2 to C7, C1 to C9, D25 to D1, D5 to D10, D9 to D11, D10 to D12, D11 to D13, D12 to D14, D27 to D15, D13 to D16, D14 to D17, D15 to D18, D16 to D19, D28 to D20, D17 to D21, D18 to D22, D19 to D23, D20 to D24, D29 to D25, D22 to D26, D23 to D27, D24 to D28, D21 to D29, D1 to D5, D26 to D6, D6 to D7, D7 to D8, D8 to D9, SW13 to SW1, SW8 to SW10, SW15 to SW11, SW9 to SW12, SW10 to SW13, SW11 to SW14, SW12 to SW15, SW1 to SW2, SW2 to SW3, SW3 to SW4, SW4 to SW5, SW14 to SW6, SW5 to SW7, SW6 to SW8, SW7 to SW9, U4 to U3, U3 to U4
Connections:
- net +3.3V: now also CH2.1 (VCC)
- net CH32V003_SWDIO: now also CH2.2 (SWDIO); no longer CH2.1 (SWDIO)
- net CH32V003_TXD: now also CH2.4 (TXD); no longer CH2.3 (TXD)
- net COL1: now also U2.19 (PD2/ADC3); no longer U2.10 (PC0)
- net COL2: now also U2.17 (PC7/SPI_MISO); no longer U2.19 (PD2/ADC3)
- net COL3: now also U2.16 (PC6/SPI_MOSI); no longer U2.17 (PC7/SPI_MISO)
- net COL4: now also U2.15 (PC5/SPI_SCK); no longer U2.16 (PC6/SPI_MOSI)
- net COL5: now also U2.13 (PC3); no longer U2.15 (PC5/SPI_SCK)
- net GND: now also CH2.3 (GND); no longer CH2.2 (GND)
